Commit message: reorganization pt2 + README

File: robot/Main Body URDF/gray.urdf (robot description, URDF)
Before this commit: robot Main Body URDF, 13 links, 12 joints
Links:
- link base_link: geometry collision mesh filename=meshes/base_link.STL; visual mesh filename=meshes/base_link.STL
- link bl_bottom: geometry collision mesh filename=meshes/bl_bottom.STL; visual mesh filename=meshes/bl_bottom.STL
- link bl_hip: geometry collision mesh filename=meshes/bl_hip.STL; visual mesh filename=meshes/bl_hip.STL
- link bl_top: geometry collision mesh filename=meshes/bl_top.STL; visual mesh filename=meshes/bl_top.STL
- link br_bottom: geometry collision mesh filename=meshes/br_bottom.STL; visual mesh filename=meshes/br_bottom.STL
- link br_hip: geometry collision mesh filename=meshes/br_hip.STL; visual mesh filename=meshes/br_hip.STL
- link br_top: geometry collision mesh filename=meshes/br_top.STL; visual mesh filename=meshes/br_top.STL
- link fl_bottom: geometry collision mesh filename=meshes/fl_bottom.STL; visual mesh filename=meshes/fl_bottom.STL
- link fl_hip: geometry collision mesh filename=meshes/fl_hip.STL; visual mesh filename=meshes/fl_hip.STL
- link fl_top: geometry collision mesh filename=meshes/fl_top.STL; visual mesh filename=meshes/fl_top.STL
- link fr_bottom: geometry collision mesh filename=meshes/fr_bottom.STL; visual mesh filename=meshes/fr_bottom.STL
- link fr_hip: geometry collision mesh filename=meshes/fr_hip.STL; visual mesh filename=meshes/fr_hip.STL
- link fr_top: geometry collision mesh filename=meshes/fr_top.STL; visual mesh filename=meshes/fr_top.STL
